Commit message: Modificado nome do arquivo urdf

File: urdf/quanser.urdf (robot description, URDF)
Before this commit: robot mob, 8 links, 8 joints
Links:
- removed link mob_origin
- added link quanser_origin

Commit message: link origin renomeado

File: urdf/quanser.urdf (robot description, URDF)
Before this commit: robot quanser, 8 links, 8 joints
Joints:
- joint chassis_joint: parent mob_origin -> quanser_origin

Commit message: Origens das juntas ajustadas

File: urdf/quanser.urdf (robot description, URDF)
Before this commit: robot quanser, 3 links, 2 joints
Joints:
- joint joint_bloco_link1: origin xyz=0.12 0.0 0.0 rpy=0 0 0 -> xyz=0.28 0.00 0.00 rpy=1.57 0 0
- joint joint_link1_link2: origin xyz=0.12 0.0 0.0 rpy=0 0 0 -> xyz=0.28 0.0 0.0 rpy=0 0 0

Commit message: bloco modificado

File: urdf/quanser.urdf (robot description, URDF)
Before this commit: robot quanser, 3 links, 2 joints
Links:
- link bloco: geometry collision box size=0.12 0.2 0.24; visual box size=0.12 0.2 0.24
Joints:
- joint joint_bloco_link1: limit lower=-1.52 upper=1.52 effort=30 velocity=1.0 -> lower=-1.57 upper=1.57 effort=30 velocity=1.0; origin xyz=0.28 0.00 0.00 rpy=1.57 0 0 -> xyz=0.18 0.00 0.00 rpy=1.57 0 0
- joint joint_link1_link2: limit lower=-1.52 upper=1.52 effort=30 velocity=1.0 -> lower=-1.57 upper=1.57 effort=30 velocity=1.0; origin xyz=0.28 0.0 0.0 rpy=0 0 0 -> xyz=0.18 0.0 0.0 rpy=0 0 0

Commit message: com bloco ajustado

File: urdf/quanser.urdf (robot description, URDF)
Before this commit: robot quanser, 3 links, 2 joints
Joints:
- joint joint_bloco_link1: origin xyz=0.18 0.00 0.00 rpy=1.57 0 0 -> xyz=0.23 0.00 0.00 rpy=1.57 0 0
- joint joint_link1_link2: origin xyz=0.18 0.0 0.0 rpy=0 0 0 -> xyz=0.3 0.0 0.0 rpy=0 0 0

Commit message: nomes adicionados

File: urdf/quanser.urdf (robot description, URDF)
Before this commit: robot quanser, 3 links, 2 joints
Links:
- link link1: geometry collision box size=0.343 0.05 0.08; visual box size=0.343 0.05 0.08
- link link2: geometry collision box size=0.267 0.05 0.08; visual box size=0.267 0.05 0.08

Commit message: Ajustes finais para submissao

File: urdf/quanser.urdf (robot description, URDF)
Before this commit: robot quanser, 3 links, 2 joints
Links:
- link link1: geometry collision box size=0.343 0.08 0.05; visual box size=0.343 0.08 0.05
- link link2: geometry collision box size=0.267 0.08 0.05; visual box size=0.267 0.08 0.05
